File: Electronics/RadioManager/RadioManager.sch (KiCad schematic (older format))
At the start: 0 parts

Commit message: Switch external interface placeholders
Parts:
- added J? (x5): CONN-8, ~, symbol CONN-8
- added J?: CONN-DC, ~, symbol CONN-DC
Connections:
- net labels added: +24V, +BATT, GND
- wire segments 0 -> 10
Changed lines of the file:
@@
 Sheet 1 1
 Title ""
-Date "23 jul 2014"
+Date "25 jul 2014"
 Rev ""
 Comp ""
@@
 Comment4 ""
 $EndDescr
+$Comp
+L CONN-8 J?
+U 1 1 53D1C0DE
+P 1100 1250
+F 0 "J?" H 1100 1700 60  0000 C CNN
+F 1 "CONN-8" H 1100 800 60  0000 C CNN
+F 2 "~" H 1100 1250 60  0000 C CNN
+F 3 "~" H 1100 1250 60  0000 C CNN
+	1    1100 1250
+	1    0    0    -1
+$EndComp
+$Comp
+L CONN-8 J?
+U 1 1 53D1C0F2
+P 1100 2550
+F 0 "J?" H 1100 3000 60  0000 C CNN
+F 1 "CONN-8" H 1100 2100 60  0000 C CNN
+F 2 "~" H 1100 2550 60  0000 C CNN
+F 3 "~" H 1100 2550 60  0000 C CNN
+	1    1100 2550
+	1    0    0    -1
+$EndComp
+$Comp
+L CONN-8 J?
+U 1 1 53D1C104
+P 1100 3650
+F 0 "J?" H 1100 4100 60  0000 C CNN
+F 1 "CONN-8" H 1100 3200 60  0000 C CNN
+F 2 "~" H 1100 3650 60  0000 C CNN
+F 3 "~" H 1100 3650 60  0000 C CNN
+	1    1100 3650
+	1    0    0    -1
+$EndComp
+$Comp
+L CONN-8 J?
+U 1 1 53D1C113
+P 1100 4750
+F 0 "J?" H 1100 5200 60  0000 C CNN
+F 1 "CONN-8" H 1100 4300 60  0000 C CNN
+F 2 "~" H 1100 4750 60  0000 C CNN
+F 3 "~" H 1100 4750 60  0000 C CNN
+	1    1100 4750
+	1    0    0    -1
+$EndComp
+$Comp
+L CONN-8 J?
+U 1 1 53D1C122
+P 1100 5850
+F 0 "J?" H 1100 6300 60  0000 C CNN
+F 1 "CONN-8" H 1100 5400 60  0000 C CNN
+F 2 "~" H 1100 5850 60  0000 C CNN
+F 3 "~" H 1100 5850 60  0000 C CNN
+	1    1100 5850
+	1    0    0    -1
+$EndComp
+$Comp
+L CONN-DC J?
+U 1 1 53D1C14A
+P 1200 6850
+F 0 "J?" H 1200 7000 60  0000 C CNN
+F 1 "CONN-DC" H 1200 6700 60  0000 C CNN
+F 2 "~" H 1200 6850 60  0000 C CNN
+F 3 "~" H 1200 6850 60  0000 C CNN
+	1    1200 6850
+	1    0    0    -1
+$EndComp
+$Comp
+L +BATT #PWR?
+U 1 1 53D1C189
+P 1600 6700
+F 0 "#PWR?" H 1600 6650 20  0001 C CNN
+F 1 "+BATT" H 1600 6800 30  0000 C CNN
+F 2 "" H 1600 6700 60  0000 C CNN
+F 3 "" H 1600 6700 60  0000 C CNN
+	1    1600 6700
+	1    0    0    -1
+$EndComp
+$Comp
+L GND #PWR?
+U 1 1 53D1C198
+P 1600 7000
+F 0 "#PWR?" H 1600 7000 30  0001 C CNN
+F 1 "GND" H 1600 6930 30  0001 C CNN
+F 2 "" H 1600 7000 60  0000 C CNN
+F 3 "" H 1600 7000 60  0000 C CNN
+	1    1600 7000
+	1    0    0    -1
+$EndComp
+Wire Wire Line
+	1600 7000 1600 6900
+Wire Wire Line
+	1600 6900 1500 6900
+Wire Wire Line
+	1500 6800 1600 6800
+Wire Wire Line
+	1600 6800 1600 6700
+$Comp
+L +24V #PWR?
+U 1 1 53D1C1B4
+P 1600 800
+F 0 "#PWR?" H 1600 750 20  0001 C CNN
+F 1 "+24V" H 1600 900 30  0000 C CNN
+F 2 "" H 1600 800 60  0000 C CNN
+F 3 "" H 1600 800 60  0000 C CNN
+	1    1600 800
+	1    0    0    -1
+$EndComp
+$Comp
+L GND #PWR?
+U 1 1 53D1C1EC
+P 1600 1700
+F 0 "#PWR?" H 1600 1700 30  0001 C CNN
+F 1 "GND" H 1600 1630 30  0001 C CNN
+F 2 "" H 1600 1700 60  0000 C CNN
+F 3 "" H 1600 1700 60  0000 C CNN
+	1    1600 1700
+	1    0    0    -1
+$EndComp
+Wire Wire Line
+	1500 1500 1600 1500
+Wire Wire Line
+	1600 1500 1600 1700
+Wire Wire Line
+	1500 1600 1600 1600
+Connection ~ 1600 1600
+Wire Wire Line
+	1600 800  1600 1300
+Wire Wire Line
+	1600 1300 1500 1300
+Wire Wire Line
+	1500 1200 1600 1200
+Connection ~ 1600 1200
 $EndSCHEMATC

Commit message: Add radio power skeleton
Parts:
- added C? (x3): C, ~, symbol C
- added D?: DIODE-SCH, ~, symbol DIODE-SCH
- added L?: L, ~, symbol L
- added R? (x2): R, ~, symbol R
- added U?: SC4503, symbol SC4503
Connections:
- wire segments 10 -> 29
Changed lines of the file:
@@
 Sheet 1 1
 Title ""
-Date "25 jul 2014"
+Date "4 aug 2014"
 Rev ""
 Comp ""
@@
 	1500 1200 1600 1200
 Connection ~ 1600 1200
+$Comp
+L SC4503 U?
+U 1 1 53DFD1D2
+P 5650 3900
+F 0 "U?" H 5650 4200 60  0000 C CNN
+F 1 "SC4503" H 5650 3600 60  0000 C CNN
+F 2 "" H 5650 3900 60  0000 C CNN
+F 3 "" H 5650 3900 60  0000 C CNN
+	1    5650 3900
+	1    0    0    -1
+$EndComp
+$Comp
+L L L?
+U 1 1 53DFD1E1
+P 5650 3400
+F 0 "L?" H 5650 3300 60  0000 C CNN
+F 1 "L" H 5650 3450 60  0000 C CNN
+F 2 "~" H 5650 3400 60  0000 C CNN
+F 3 "~" H 5650 3400 60  0000 C CNN
+	1    5650 3400
+	1    0    0    -1
+$EndComp
+$Comp
+L DIODE-SCH D?
+U 1 1 53DFD1F0
+P 6550 3400
+F 0 "D?" H 6550 3500 60  0000 C CNN
+F 1 "DIODE-SCH" H 6550 3300 60  0000 C CNN
+F 2 "~" H 6550 3400 60  0000 C CNN
+F 3 "~" H 6550 3400 60  0000 C CNN
+	1    6550 3400
+	1    0    0    -1
+$EndComp
+$Comp
+L R R?
+U 1 1 53DFD5A4
+P 7400 3750
+F 0 "R?" H 7400 3850 50  0000 C CNN
+F 1 "R" H 7400 3750 50  0000 C CNN
+F 2 "~" H 7400 3750 60  0000 C CNN
+F 3 "~" H 7400 3750 60  0000 C CNN
+F 4 "W" H 7400 3650 50  0001 C CNN "Power"
+F 5 "%" H 7400 3550 50  0001 C CNN "Tolerance"
+	1    7400 3750
+	0    1    -1   0
+$EndComp
+$Comp
+L R R?
+U 1 1 53DFD5C6
+P 7400 4450
+F 0 "R?" H 7400 4550 50  0000 C CNN
+F 1 "R" H 7400 4450 50  0000 C CNN
+F 2 "~" H 7400 4450 60  0000 C CNN
+F 3 "~" H 7400 4450 60  0000 C CNN
+F 4 "W" H 7400 4350 50  0001 C CNN "Power"
+F 5 "%" H 7400 4250 50  0001 C CNN "Tolerance"
+	1    7400 4450
+	0    1    -1   0
+$EndComp
+$Comp
+L C C?
+U 1 1 53DFD5E1
+P 7100 3750
+F 0 "C?" H 7150 3900 60  0000 L CNN
+F 1 "C" H 7150 3600 60  0000 L CNN
+F 2 "~" H 7100 3750 60  0000 C CNN
+F 3 "~" H 7100 3750 60  0000 C CNN
+F 4 "V" H 7050 3600 60  0001 R CNN "Voltage"
+F 5 "D" H 7050 3900 60  0001 R CNN "Dielectric"
+	1    7100 3750
+	-1   0    0    -1
+$EndComp
+Wire Wire Line
+	6100 4100 7400 4100
+Wire Wire Line
+	7400 4000 7400 4200
+Connection ~ 7400 4100
+Wire Wire Line
+	6800 3400 7700 3400
+Wire Wire Line
+	7400 3400 7400 3500
+Wire Wire Line
+	5900 3400 6300 3400
+Wire Wire Line
+	6100 3700 6200 3700
+Wire Wire Line
+	6200 3700 6200 3400
+Connection ~ 6200 3400
+Wire Wire Line
+	7100 3500 7100 3400
+Connection ~ 7100 3400
+Wire Wire Line
+	7100 4000 7100 4100
+Connection ~ 7100 4100
+$Comp
+L C C?
+U 1 1 53DFD69D
+P 7700 3750
+F 0 "C?" H 7750 3900 60  0000 L CNN
+F 1 "C" H 7750 3600 60  0000 L CNN
+F 2 "~" H 7700 3750 60  0000 C CNN
+F 3 "~" H 7700 3750 60  0000 C CNN
+F 4 "V" H 7650 3600 60  0001 R CNN "Voltage"
+F 5 "D" H 7650 3900 60  0001 R CNN "Dielectric"
+	1    7700 3750
+	1    0    0    -1
+$EndComp
+Wire Wire Line
+	7700 3300 7700 3500
+Connection ~ 7400 3400
+$Comp
+L +24V #PWR?
+U 1 1 53DFD6D2
+P 7700 3300
+F 0 "#PWR?" H 7700 3250 20  0001 C CNN
+F 1 "+24V" H 7700 3400 30  0000 C CNN
+F 2 "" H 7700 3300 60  0000 C CNN
+F 3 "" H 7700 3300 60  0000 C CNN
+	1    7700 3300
+	1    0    0    -1
+$EndComp
+Connection ~ 7700 3400
+$Comp
+L GND #PWR?
+U 1 1 53DFD6FD
+P 7700 4100
+F 0 "#PWR?" H 7700 4100 30  0001 C CNN
+F 1 "GND" H 7700 4030 30  0001 C CNN
+F 2 "" H 7700 4100 60  0000 C CNN
+F 3 "" H 7700 4100 60  0000 C CNN
+	1    7700 4100
+	1    0    0    -1
+$EndComp
+$Comp
+L GND #PWR?
+U 1 1 53DFD70C
+P 7400 4800
+F 0 "#PWR?" H 7400 4800 30  0001 C CNN
+F 1 "GND" H 7400 4730 30  0001 C CNN
+F 2 "" H 7400 4800 60  0000 C CNN
+F 3 "" H 7400 4800 60  0000 C CNN
+	1    7400 4800
+	1    0    0    -1
+$EndComp
+$Comp
+L GND #PWR?
+U 1 1 53DFD71B
+P 5100 4200
+F 0 "#PWR?" H 5100 4200 30  0001 C CNN
+F 1 "GND" H 5100 4130 30  0001 C CNN
+F 2 "" H 5100 4200 60  0000 C CNN
+F 3 "" H 5100 4200 60  0000 C CNN
+	1    5100 4200
+	1    0    0    -1
+$EndComp
+Wire Wire Line
+	5100 4200 5100 4100
+Wire Wire Line
+	5100 4100 5200 4100
+Wire Wire Line
+	7700 4000 7700 4100
+Wire Wire Line
+	7400 4700 7400 4800
+$Comp
+L +BATT #PWR?
+U 1 1 53DFD786
+P 4400 3300
+F 0 "#PWR?" H 4400 3250 20  0001 C CNN
+F 1 "+BATT" H 4400 3400 30  0000 C CNN
+F 2 "" H 4400 3300 60  0000 C CNN
+F 3 "" H 4400 3300 60  0000 C CNN
+	1    4400 3300
+	1    0    0    -1
+$EndComp
+Wire Wire Line
+	4400 3300 4400 3500
+Wire Wire Line
+	4400 3400 5400 3400
+$Comp
+L C C?
+U 1 1 53DFD7B6
+P 4400 3750
+F 0 "C?" H 4450 3900 60  0000 L CNN
+F 1 "C" H 4450 3600 60  0000 L CNN
+F 2 "~" H 4400 3750 60  0000 C CNN
+F 3 "~" H 4400 3750 60  0000 C CNN
+F 4 "V" H 4350 3600 60  0001 R CNN "Voltage"
+F 5 "D" H 4350 3900 60  0001 R CNN "Dielectric"
+	1    4400 3750
+	-1   0    0    -1
+$EndComp
+$Comp
+L GND #PWR?
+U 1 1 53DFD7D1
+P 4400 4100
+F 0 "#PWR?" H 4400 4100 30  0001 C CNN
+F 1 "GND" H 4400 4030 30  0001 C CNN
+F 2 "" H 4400 4100 60  0000 C CNN
+F 3 "" H 4400 4100 60  0000 C CNN
+	1    4400 4100
+	1    0    0    -1
+$EndComp
+Wire Wire Line
+	4400 4100 4400 4000
+Connection ~ 4400 3400
+Wire Wire Line
+	5200 3700 5100 3700
+Wire Wire Line
+	5100 3700 5100 3400
+Connection ~ 5100 3400
 $EndSCHEMATC

Commit message: Add switch datasheet and sheet
Parts:
- added C?: C, ~, symbol C
- added R?: R, ~, symbol R
Connections:
- net labels added: RADIO_EN
- wire segments 29 -> 35
Other:
- moved on the sheet: C?
Changed lines of the file:
@@
 $Descr A4 11693 8268
 encoding utf-8
-Sheet 1 1
+Sheet 1 2
 Title ""
 Date "4 aug 2014"
@@
 L +BATT #PWR?
 U 1 1 53DFD786
-P 4400 3300
-F 0 "#PWR?" H 4400 3250 20  0001 C CNN
-F 1 "+BATT" H 4400 3400 30  0000 C CNN
-F 2 "" H 4400 3300 60  0000 C CNN
-F 3 "" H 4400 3300 60  0000 C CNN
-	1    4400 3300
-	1    0    0    -1
-$EndComp
-Wire Wire Line
-	4400 3300 4400 3500
-Wire Wire Line
-	4400 3400 5400 3400
+P 4100 3300
+F 0 "#PWR?" H 4100 3250 20  0001 C CNN
+F 1 "+BATT" H 4100 3400 30  0000 C CNN
+F 2 "" H 4100 3300 60  0000 C CNN
+F 3 "" H 4100 3300 60  0000 C CNN
+	1    4100 3300
+	1    0    0    -1
+$EndComp
+Wire Wire Line
+	4100 3300 4100 3500
+Wire Wire Line
+	4100 3400 5400 3400
 $Comp
 L C C?
 U 1 1 53DFD7B6
-P 4400 3750
-F 0 "C?" H 4450 3900 60  0000 L CNN
-F 1 "C" H 4450 3600 60  0000 L CNN
-F 2 "~" H 4400 3750 60  0000 C CNN
-F 3 "~" H 4400 3750 60  0000 C CNN
-F 4 "V" H 4350 3600 60  0001 R CNN "Voltage"
-F 5 "D" H 4350 3900 60  0001 R CNN "Dielectric"
-	1    4400 3750
+P 4100 3750
+F 0 "C?" H 4150 3900 60  0000 L CNN
+F 1 "C" H 4150 3600 60  0000 L CNN
+F 2 "~" H 4100 3750 60  0000 C CNN
+F 3 "~" H 4100 3750 60  0000 C CNN
+F 4 "V" H 4050 3600 60  0001 R CNN "Voltage"
+F 5 "D" H 4050 3900 60  0001 R CNN "Dielectric"
+	1    4100 3750
 	-1   0    0    -1
 $EndComp
@@
 L GND #PWR?
 U 1 1 53DFD7D1
-P 4400 4100
-F 0 "#PWR?" H 4400 4100 30  0001 C CNN
-F 1 "GND" H 4400 4030 30  0001 C CNN
-F 2 "" H 4400 4100 60  0000 C CNN
-F 3 "" H 4400 4100 60  0000 C CNN
-	1    4400 4100
-	1    0    0    -1
-$EndComp
-Wire Wire Line
-	4400 4100 4400 4000
-Connection ~ 4400 3400
+P 4100 4100
+F 0 "#PWR?" H 4100 4100 30  0001 C CNN
+F 1 "GND" H 4100 4030 30  0001 C CNN
+F 2 "" H 4100 4100 60  0000 C CNN
+F 3 "" H 4100 4100 60  0000 C CNN
+	1    4100 4100
+	1    0    0    -1
+$EndComp
+Wire Wire Line
+	4100 4100 4100 4000
+Connection ~ 4100 3400
 Wire Wire Line
 	5200 3700 5100 3700
@@
 	5100 3700 5100 3400
 Connection ~ 5100 3400
+$Comp
+L C C?
+U 1 1 53DFD8DE
+P 4800 4250
+F 0 "C?" H 4850 4400 60  0000 L CNN
+F 1 "C" H 4850 4100 60  0000 L CNN
+F 2 "~" H 4800 4250 60  0000 C CNN
+F 3 "~" H 4800 4250 60  0000 C CNN
+F 4 "V" H 4750 4100 60  0001 R CNN "Voltage"
+F 5 "D" H 4750 4400 60  0001 R CNN "Dielectric"
+	1    4800 4250
+	-1   0    0    -1
+$EndComp
+$Comp
+L R R?
+U 1 1 53DFD8E6
+P 4400 4250
+F 0 "R?" H 4400 4350 50  0000 C CNN
+F 1 "R" H 4400 4250 50  0000 C CNN
+F 2 "~" H 4400 4250 60  0000 C CNN
+F 3 "~" H 4400 4250 60  0000 C CNN
+F 4 "W" H 4400 4150 50  0001 C CNN "Power"
+F 5 "%" H 4400 4050 50  0001 C CNN "Tolerance"
+	1    4400 4250
+	0    -1   -1   0
+$EndComp
+Wire Wire Line
+	4400 4000 4400 3900
+Wire Wire Line
+	4400 3900 5200 3900
+Wire Wire Line
+	4800 4000 4800 3900
+Connection ~ 4800 3900
+$Comp
+L GND #PWR?
+U 1 1 53DFD975
+P 4800 4600
+F 0 "#PWR?" H 4800 4600 30  0001 C CNN
+F 1 "GND" H 4800 4530 30  0001 C CNN
+F 2 "" H 4800 4600 60  0000 C CNN
+F 3 "" H 4800 4600 60  0000 C CNN
+	1    4800 4600
+	1    0    0    -1
+$EndComp
+Wire Wire Line
+	4800 4500 4800 4600
+Text Label 4300 4600 2    60   ~ 0
+RADIO_EN
+Wire Wire Line
+	4300 4600 4400 4600
+Wire Wire Line
+	4400 4600 4400 4500
+$Sheet
+S 5600 1800 1000 1000
+U 53DFFD33
+F0 "Switch" 50
+F1 "Switch.sch" 50
+$EndSheet
 $EndSCHEMATC

Commit message: Add actual RJ45 jacks
Parts:
- removed J? (x5): CONN-8, ~, symbol CONN-8
- added J? (x10): RJ45-MAG-LED, symbol RJ45-MAG-LED
Connections:
- wire segments 35 -> 29
Changed lines of the file:
@@
 Sheet 1 2
 Title ""
-Date "4 aug 2014"
+Date "10 sep 2014"
 Rev ""
 Comp ""
@@
 Comment4 ""
 $EndDescr
-$Comp
-L CONN-8 J?
-U 1 1 53D1C0DE
-P 1100 1250
-F 0 "J?" H 1100 1700 60  0000 C CNN
-F 1 "CONN-8" H 1100 800 60  0000 C CNN
-F 2 "~" H 1100 1250 60  0000 C CNN
-F 3 "~" H 1100 1250 60  0000 C CNN
-	1    1100 1250
-	1    0    0    -1
-$EndComp
-$Comp
-L CONN-8 J?
-U 1 1 53D1C0F2
-P 1100 2550
-F 0 "J?" H 1100 3000 60  0000 C CNN
-F 1 "CONN-8" H 1100 2100 60  0000 C CNN
-F 2 "~" H 1100 2550 60  0000 C CNN
-F 3 "~" H 1100 2550 60  0000 C CNN
-	1    1100 2550
-	1    0    0    -1
-$EndComp
-$Comp
-L CONN-8 J?
-U 1 1 53D1C104
-P 1100 3650
-F 0 "J?" H 1100 4100 60  0000 C CNN
-F 1 "CONN-8" H 1100 3200 60  0000 C CNN
-F 2 "~" H 1100 3650 60  0000 C CNN
-F 3 "~" H 1100 3650 60  0000 C CNN
-	1    1100 3650
-	1    0    0    -1
-$EndComp
-$Comp
-L CONN-8 J?
-U 1 1 53D1C113
-P 1100 4750
-F 0 "J?" H 1100 5200 60  0000 C CNN
-F 1 "CONN-8" H 1100 4300 60  0000 C CNN
-F 2 "~" H 1100 4750 60  0000 C CNN
-F 3 "~" H 1100 4750 60  0000 C CNN
-	1    1100 4750
-	1    0    0    -1
-$EndComp
-$Comp
-L CONN-8 J?
-U 1 1 53D1C122
-P 1100 5850
-F 0 "J?" H 1100 6300 60  0000 C CNN
-F 1 "CONN-8" H 1100 5400 60  0000 C CNN
-F 2 "~" H 1100 5850 60  0000 C CNN
-F 3 "~" H 1100 5850 60  0000 C CNN
-	1    1100 5850
-	1    0    0    -1
-$EndComp
 $Comp
 L CONN-DC J?
@@
 Wire Wire Line
 	1600 6800 1600 6700
-$Comp
-L +24V #PWR?
-U 1 1 53D1C1B4
-P 1600 800
-F 0 "#PWR?" H 1600 750 20  0001 C CNN
-F 1 "+24V" H 1600 900 30  0000 C CNN
-F 2 "" H 1600 800 60  0000 C CNN
-F 3 "" H 1600 800 60  0000 C CNN
-	1    1600 800
-	1    0    0    -1
-$EndComp
-$Comp
-L GND #PWR?
-U 1 1 53D1C1EC
-P 1600 1700
-F 0 "#PWR?" H 1600 1700 30  0001 C CNN
-F 1 "GND" H 1600 1630 30  0001 C CNN
-F 2 "" H 1600 1700 60  0000 C CNN
-F 3 "" H 1600 1700 60  0000 C CNN
-	1    1600 1700
-	1    0    0    -1
-$EndComp
-Wire Wire Line
-	1500 1500 1600 1500
-Wire Wire Line
-	1600 1500 1600 1700
-Wire Wire Line
-	1500 1600 1600 1600
-Connection ~ 1600 1600
-Wire Wire Line
-	1600 800  1600 1300
-Wire Wire Line
-	1600 1300 1500 1300
-Wire Wire Line
-	1500 1200 1600 1200
-Connection ~ 1600 1200
 $Comp
 L SC4503 U?
@@
 F1 "Switch.sch" 50
 $EndSheet
+$Comp
+L RJ45-MAG-LED J?
+U 1 1 540FBEAD
+P 1150 1300
+F 0 "J?" H 1150 1800 60  0000 C CNN
+F 1 "RJ45-MAG-LED" V 1350 1300 60  0000 C CNN
+F 2 "" H 1150 1300 60  0000 C CNN
+F 3 "" H 1150 1300 60  0000 C CNN
+F 4 "Bel Fuse" H 1150 1300 60  0001 C CNN "MFR Name"
+F 5 "0826-1L1T-57-F" H 1150 1300 60  0001 C CNN "MFR Part No"
+F 6 "507-1431-ND" H 1150 1300 60  0001 C CNN "Distributor Part No"
+	1    1150 1300
+	-1   0    0    -1
+$EndComp
+$Comp
+L RJ45-MAG-LED J?
+U 2 1 540FBEE7
+P 1950 1300
+F 0 "J?" H 1950 1800 60  0000 C CNN
+F 1 "RJ45-MAG-LED" V 2150 1300 60  0000 C CNN
+F 2 "" H 1950 1300 60  0000 C CNN
+F 3 "" H 1950 1300 60  0000 C CNN
+F 4 "Bel Fuse" H 1950 1300 60  0001 C CNN "MFR Name"
+F 5 "0826-1L1T-57-F" H 1950 1300 60  0001 C CNN "MFR Part No"
+F 6 "507-1431-ND" H 1950 1300 60  0001 C CNN "Distributor Part No"
+	2    1950 1300
+	-1   0    0    -1
+$EndComp
+$Comp
+L RJ45-MAG-LED J?
+U 1 1 540FBEF8
+P 1150 2400
+F 0 "J?" H 1150 2900 60  0000 C CNN
+F 1 "RJ45-MAG-LED" V 1350 2400 60  0000 C CNN
+F 2 "" H 1150 2400 60  0000 C CNN
+F 3 "" H 1150 2400 60  0000 C CNN
+F 4 "Bel Fuse" H 1150 2400 60  0001 C CNN "MFR Name"
+F 5 "0826-1L1T-57-F" H 1150 2400 60  0001 C CNN "MFR Part No"
+F 6 "507-1431-ND" H 1150 2400 60  0001 C CNN "Distributor Part No"
+	1    1150 2400
+	-1   0    0    -1
+$EndComp
+$Comp
+L RJ45-MAG-LED J?
+U 2 1 540FBF01
+P 1950 2400
+F 0 "J?" H 1950 2900 60  0000 C CNN
+F 1 "RJ45-MAG-LED" V 2150 2400 60  0000 C CNN
+F 2 "" H 1950 2400 60  0000 C CNN
+F 3 "" H 1950 2400 60  0000 C CNN
+F 4 "Bel Fuse" H 1950 2400 60  0001 C CNN "MFR Name"
+F 5 "0826-1L1T-57-F" H 1950 2400 60  0001 C CNN "MFR Part No"
+F 6 "507-1431-ND" H 1950 2400 60  0001 C CNN "Distributor Part No"
+	2    1950 2400
+	-1   0    0    -1
+$EndComp
+$Comp
+L RJ45-MAG-LED J?
+U 1 1 540FBF0A
+P 1150 3500
+F 0 "J?" H 1150 4000 60  0000 C CNN
+F 1 "RJ45-MAG-LED" V 1350 3500 60  0000 C CNN
+F 2 "" H 1150 3500 60  0000 C CNN
+F 3 "" H 1150 3500 60  0000 C CNN
+F 4 "Bel Fuse" H 1150 3500 60  0001 C CNN "MFR Name"
+F 5 "0826-1L1T-57-F" H 1150 3500 60  0001 C CNN "MFR Part No"
+F 6 "507-1431-ND" H 1150 3500 60  0001 C CNN "Distributor Part No"
+	1    1150 3500
+	-1   0    0    -1
+$EndComp
+$Comp
+L RJ45-MAG-LED J?
+U 2 1 540FBF13
+P 1950 3500
+F 0 "J?" H 1950 4000 60  0000 C CNN
+F 1 "RJ45-MAG-LED" V 2150 3500 60  0000 C CNN
+F 2 "" H 1950 3500 60  0000 C CNN
+F 3 "" H 1950 3500 60  0000 C CNN
+F 4 "Bel Fuse" H 1950 3500 60  0001 C CNN "MFR Name"
+F 5 "0826-1L1T-57-F" H 1950 3500 60  0001 C CNN "MFR Part No"
+F 6 "507-1431-ND" H 1950 3500 60  0001 C CNN "Distributor Part No"
+	2    1950 3500
+	-1   0    0    -1
+$EndComp
+$Comp
+L RJ45-MAG-LED J?
+U 1 1 540FBF1C
+P 1150 4600
+F 0 "J?" H 1150 5100 60  0000 C CNN
+F 1 "RJ45-MAG-LED" V 1350 4600 60  0000 C CNN
+F 2 "" H 1150 4600 60  0000 C CNN
+F 3 "" H 1150 4600 60  0000 C CNN
+F 4 "Bel Fuse" H 1150 4600 60  0001 C CNN "MFR Name"
+F 5 "0826-1L1T-57-F" H 1150 4600 60  0001 C CNN "MFR Part No"
+F 6 "507-1431-ND" H 1150 4600 60  0001 C CNN "Distributor Part No"
+	1    1150 4600
+	-1   0    0    -1
+$EndComp
+$Comp
+L RJ45-MAG-LED J?
+U 2 1 540FBF25
+P 1950 4600
+F 0 "J?" H 1950 5100 60  0000 C CNN
+F 1 "RJ45-MAG-LED" V 2150 4600 60  0000 C CNN
+F 2 "" H 1950 4600 60  0000 C CNN
+F 3 "" H 1950 4600 60  0000 C CNN
+F 4 "Bel Fuse" H 1950 4600 60  0001 C CNN "MFR Name"
+F 5 "0826-1L1T-57-F" H 1950 4600 60  0001 C CNN "MFR Part No"
+F 6 "507-1431-ND" H 1950 4600 60  0001 C CNN "Distributor Part No"
+	2    1950 4600
+	-1   0    0    -1
+$EndComp
+$Comp
+L RJ45-MAG-LED J?
+U 1 1 540FBF2E
+P 1150 5700
+F 0 "J?" H 1150 6200 60  0000 C CNN
+F 1 "RJ45-MAG-LED" V 1350 5700 60  0000 C CNN
+F 2 "" H 1150 5700 60  0000 C CNN
+F 3 "" H 1150 5700 60  0000 C CNN
+F 4 "Bel Fuse" H 1150 5700 60  0001 C CNN "MFR Name"
+F 5 "0826-1L1T-57-F" H 1150 5700 60  0001 C CNN "MFR Part No"
+F 6 "507-1431-ND" H 1150 5700 60  0001 C CNN "Distributor Part No"
+	1    1150 5700
+	-1   0    0    -1
+$EndComp
+$Comp
+L RJ45-MAG-LED J?
+U 2 1 540FBF37
+P 1950 5700
+F 0 "J?" H 1950 6200 60  0000 C CNN
+F 1 "RJ45-MAG-LED" V 2150 5700 60  0000 C CNN
+F 2 "" H 1950 5700 60  0000 C CNN
+F 3 "" H 1950 5700 60  0000 C CNN
+F 4 "Bel Fuse" H 1950 5700 60  0001 C CNN "MFR Name"
+F 5 "0826-1L1T-57-F" H 1950 5700 60  0001 C CNN "MFR Part No"
+F 6 "507-1431-ND" H 1950 5700 60  0001 C CNN "Distributor Part No"
+	2    1950 5700
+	-1   0    0    -1
+$EndComp
 $EndSCHEMATC
