File: Electronics/RadioManager/Power.sch (KiCad schematic (older format))
At the start: 28 parts, among them U2 SC4503, U3 AOZ1280, U4 AOZ1280

Commit message: Swap tx/rx pairs for better routing
Parts:
- C26, C27: value C -> 10000pF; Dielectric D -> X7R; Distributor Part No (none) -> 1276-1009-1-ND; MFR Name (none) -> Samsung; MFR Part No (none) -> CL10B103KB8NNNC; Voltage V -> 50V
- D1, D3, D4: value DIODE-SCH -> CDBA140; Distributor Part No (none) -> 641-1015-1-ND; MFR Name (none) -> Comchip; MFR Part No (none) -> CDBA140-G
- R12: value R -> 49.9k
- R13: value R -> 15.8k
- R14: value R -> 80.6k
- R15: value R -> 64.2k
Other:
- moved on the sheet: C20
Changed lines of the file:
@@
 $Descr A4 11693 8268
 encoding utf-8
-Sheet 3 3
+Sheet 2 3
 Title ""
-Date "22 sep 2014"
+Date "3 oct 2014"
 Rev ""
 Comp ""
@@
 F 3 "~" H 3050 1400 60  0000 C CNN
 	1    3050 1400
-	1    0    0    -1
-$EndComp
-$Comp
-L DIODE-SCH D1
-U 1 1 5410EB9F
-P 3950 1400
-F 0 "D1" H 3950 1500 60  0000 C CNN
-F 1 "DIODE-SCH" H 3950 1300 60  0000 C CNN
-F 2 "~" H 3950 1400 60  0000 C CNN
-F 3 "~" H 3950 1400 60  0000 C CNN
-	1    3950 1400
 	1    0    0    -1
 $EndComp
@@
 Connection ~ 4800 2100
 Wire Wire Line
-	4200 1400 5100 1400
+	4200 1400 5200 1400
 Wire Wire Line
 	4800 1400 4800 1500
@@
 L C C20
 U 1 1 5410EBCC
-P 5100 1750
-F 0 "C20" H 5150 1900 60  0000 L CNN
-F 1 "C" H 5150 1600 60  0000 L CNN
-F 2 "~" H 5100 1750 60  0000 C CNN
-F 3 "~" H 5100 1750 60  0000 C CNN
-F 4 "V" H 5050 1600 60  0001 R CNN "Voltage"
-F 5 "D" H 5050 1900 60  0001 R CNN "Dielectric"
-	1    5100 1750
-	1    0    0    -1
-$EndComp
-Wire Wire Line
-	5100 1300 5100 1500
+P 5200 1750
+F 0 "C20" H 5250 1900 60  0000 L CNN
+F 1 "C" H 5250 1600 60  0000 L CNN
+F 2 "~" H 5200 1750 60  0000 C CNN
+F 3 "~" H 5200 1750 60  0000 C CNN
+F 4 "V" H 5150 1600 60  0001 R CNN "Voltage"
+F 5 "D" H 5150 1900 60  0001 R CNN "Dielectric"
+	1    5200 1750
+	1    0    0    -1
+$EndComp
+Wire Wire Line
+	5200 1300 5200 1500
 Connection ~ 4800 1400
 $Comp
 L +24V #PWR012
 U 1 1 5410EBD4
-P 5100 1300
-F 0 "#PWR012" H 5100 1250 20  0001 C CNN
-F 1 "+24V" H 5100 1400 30  0000 C CNN
-F 2 "" H 5100 1300 60  0000 C CNN
-F 3 "" H 5100 1300 60  0000 C CNN
-	1    5100 1300
-	1    0    0    -1
-$EndComp
-Connection ~ 5100 1400
+P 5200 1300
+F 0 "#PWR012" H 5200 1250 20  0001 C CNN
+F 1 "+24V" H 5200 1400 30  0000 C CNN
+F 2 "" H 5200 1300 60  0000 C CNN
+F 3 "" H 5200 1300 60  0000 C CNN
+	1    5200 1300
+	1    0    0    -1
+$EndComp
+Connection ~ 5200 1400
 $Comp
 L GND #PWR013
 U 1 1 5410EBDB
-P 5100 2100
-F 0 "#PWR013" H 5100 2100 30  0001 C CNN
-F 1 "GND" H 5100 2030 30  0001 C CNN
-F 2 "" H 5100 2100 60  0000 C CNN
-F 3 "" H 5100 2100 60  0000 C CNN
-	1    5100 2100
+P 5200 2100
+F 0 "#PWR013" H 5200 2100 30  0001 C CNN
+F 1 "GND" H 5200 2030 30  0001 C CNN
+F 2 "" H 5200 2100 60  0000 C CNN
+F 3 "" H 5200 2100 60  0000 C CNN
+	1    5200 2100
 	1    0    0    -1
 $EndComp
@@
 	2500 2100 2600 2100
 Wire Wire Line
-	5100 2000 5100 2100
+	5200 2000 5200 2100
 Wire Wire Line
 	4800 2700 4800 2800
@@
 	1    0    0    -1
 $EndComp
-$Comp
-L C C27
-U 1 1 54160FBC
-P 8450 3900
-F 0 "C27" H 8500 4050 60  0000 L CNN
-F 1 "C" H 8500 3750 60  0000 L CNN
-F 2 "~" H 8450 3900 60  0000 C CNN
-F 3 "~" H 8450 3900 60  0000 C CNN
-F 4 "V" H 8400 3750 60  0001 R CNN "Voltage"
-F 5 "D" H 8400 4050 60  0001 R CNN "Dielectric"
-	1    8450 3900
-	0    -1   -1   0
-$EndComp
 Wire Wire Line
 	8200 3900 7900 3900
@@
 P 9700 4650
 F 0 "R14" H 9700 4750 50  0000 C CNN
-F 1 "R" H 9700 4650 50  0000 C CNN
+F 1 "80.6k" H 9700 4650 50  0000 C CNN
 F 2 "~" H 9700 4650 60  0000 C CNN
 F 3 "~" H 9700 4650 60  0000 C CNN
@@
 P 9700 5350
 F 0 "R15" H 9700 5450 50  0000 C CNN
-F 1 "R" H 9700 5350 50  0000 C CNN
+F 1 "64.2k" H 9700 5350 50  0000 C CNN
 F 2 "~" H 9700 5350 60  0000 C CNN
 F 3 "~" H 9700 5350 60  0000 C CNN
@@
 F 5 "%" H 9700 5150 50  0001 C CNN "Tolerance"
 	1    9700 5350
-	0    -1   -1   0
-$EndComp
-$Comp
-L DIODE-SCH D4
-U 1 1 54161067
-P 9000 4650
-F 0 "D4" H 9000 4750 60  0000 C CNN
-F 1 "DIODE-SCH" H 9000 4550 60  0000 C CNN
-F 2 "~" H 9000 4650 60  0000 C CNN
-F 3 "~" H 9000 4650 60  0000 C CNN
-	1    9000 4650
 	0    -1   -1   0
 $EndComp
@@
 P 8450 1300
 F 0 "C26" H 8500 1450 60  0000 L CNN
-F 1 "C" H 8500 1150 60  0000 L CNN
+F 1 "10000pF" H 8500 1150 60  0000 L CNN
 F 2 "~" H 8450 1300 60  0000 C CNN
 F 3 "~" H 8450 1300 60  0000 C CNN
-F 4 "V" H 8400 1150 60  0001 R CNN "Voltage"
-F 5 "D" H 8400 1450 60  0001 R CNN "Dielectric"
+F 4 "Samsung" H 8450 1300 60  0001 C CNN "MFR Name"
+F 5 "CL10B103KB8NNNC" H 8450 1300 60  0001 C CNN "MFR Part No"
+F 6 "1276-1009-1-ND" H 8450 1300 60  0001 C CNN "Distributor Part No"
+F 7 "50V" H 8400 1150 60  0001 R CNN "Voltage"
+F 8 "X7R" H 8400 1450 60  0001 R CNN "Dielectric"
 	1    8450 1300
 	0    -1   -1   0
@@
 P 9700 2050
 F 0 "R12" H 9700 2150 50  0000 C CNN
-F 1 "R" H 9700 2050 50  0000 C CNN
+F 1 "49.9k" H 9700 2050 50  0000 C CNN
 F 2 "~" H 9700 2050 60  0000 C CNN
 F 3 "~" H 9700 2050 60  0000 C CNN
@@
 P 9700 2750
 F 0 "R13" H 9700 2850 50  0000 C CNN
-F 1 "R" H 9700 2750 50  0000 C CNN
+F 1 "15.8k" H 9700 2750 50  0000 C CNN
 F 2 "~" H 9700 2750 60  0000 C CNN
 F 3 "~" H 9700 2750 60  0000 C CNN
@@
 P 9000 2050
 F 0 "D3" H 9000 2150 60  0000 C CNN
-F 1 "DIODE-SCH" H 9000 1950 60  0000 C CNN
+F 1 "CDBA140" H 9000 1950 60  0000 C CNN
 F 2 "~" H 9000 2050 60  0000 C CNN
 F 3 "~" H 9000 2050 60  0000 C CNN
+F 4 "Comchip" H 9000 2050 60  0001 C CNN "MFR Name"
+F 5 "CDBA140-G" H 9000 2050 60  0001 C CNN "MFR Part No"
+F 6 "641-1015-1-ND" H 9000 2050 60  0001 C CNN "Distributor Part No"
 	1    9000 2050
 	0    -1   -1   0
@@
 $EndComp
 Connection ~ 10100 1700
+$Comp
+L C C27
+U 1 1 542E03F3
+P 8450 3900
+F 0 "C27" H 8500 4050 60  0000 L CNN
+F 1 "10000pF" H 8500 3750 60  0000 L CNN
+F 2 "~" H 8450 3900 60  0000 C CNN
+F 3 "~" H 8450 3900 60  0000 C CNN
+F 4 "Samsung" H 8450 3900 60  0001 C CNN "MFR Name"
+F 5 "CL10B103KB8NNNC" H 8450 3900 60  0001 C CNN "MFR Part No"
+F 6 "1276-1009-1-ND" H 8450 3900 60  0001 C CNN "Distributor Part No"
+F 7 "50V" H 8400 3750 60  0001 R CNN "Voltage"
+F 8 "X7R" H 8400 4050 60  0001 R CNN "Dielectric"
+	1    8450 3900
+	0    -1   -1   0
+$EndComp
+$Comp
+L DIODE-SCH D4
+U 1 1 542E1DC4
+P 9000 4650
+F 0 "D4" H 9000 4750 60  0000 C CNN
+F 1 "CDBA140" H 9000 4550 60  0000 C CNN
+F 2 "~" H 9000 4650 60  0000 C CNN
+F 3 "~" H 9000 4650 60  0000 C CNN
+F 4 "Comchip" H 9000 4650 60  0001 C CNN "MFR Name"
+F 5 "CDBA140-G" H 9000 4650 60  0001 C CNN "MFR Part No"
+F 6 "641-1015-1-ND" H 9000 4650 60  0001 C CNN "Distributor Part No"
+	1    9000 4650
+	0    -1   -1   0
+$EndComp
+$Comp
+L DIODE-SCH D1
+U 1 1 542E1DE3
+P 3950 1400
+F 0 "D1" H 3950 1500 60  0000 C CNN
+F 1 "CDBA140" H 3950 1300 60  0000 C CNN
+F 2 "~" H 3950 1400 60  0000 C CNN
+F 3 "~" H 3950 1400 60  0000 C CNN
+F 4 "Comchip" H 3950 1400 60  0001 C CNN "MFR Name"
+F 5 "CDBA140-G" H 3950 1400 60  0001 C CNN "MFR Part No"
+F 6 "641-1015-1-ND" H 3950 1400 60  0001 C CNN "Distributor Part No"
+	1    3950 1400
+	1    0    0    -1
+$EndComp
 $EndSCHEMATC

Commit message: Resistor values
Parts:
- removed C18: C, ~, symbol C
- R1, R10, R11: value R -> 10k; Distributor Part No (none) -> RHM10KCGCT-ND; MFR Name (none) -> Rohm; MFR Part No (none) -> MCR03ERTJ103; Power W -> 1/10W; Tolerance % -> 5%
- R12: Distributor Part No (none) -> 311-49.9KHRCT-ND; MFR Name (none) -> Yageo; MFR Part No (none) -> RC0603FR-0749K9L; Power W -> 1/10W; Tolerance % -> 1%
- R13: Distributor Part No (none) -> ERJ-3EKF1582V; MFR Name (none) -> Panasonic; MFR Part No (none) -> P15.8KHCT-ND; Power W -> 1/10W; Tolerance % -> 1%
- R14: Distributor Part No (none) -> P80.6KHCT-ND; MFR Name (none) -> Panasonic; MFR Part No (none) -> ERJ-3EKF8062V; Power W -> 1/10W; Tolerance % -> 1%
- R15: value 64.2k -> 64.9k; Distributor Part No (none) -> RHM64.9KCFCT-ND; MFR Name (none) -> Rohm; MFR Part No (none) -> MCR03ERTF6492; Power W -> 1/10W; Tolerance % -> 1%
- R2: value R -> 287k; Distributor Part No (none) -> RHM287KCFCT-ND; MFR Name (none) -> Rohm; MFR Part No (none) -> MCR03ERTF2873; Power W -> 1/10W; Tolerance % -> 1%
- R3: value R -> 15.8k; Distributor Part No (none) -> ERJ-3EKF1582V; MFR Name (none) -> Panasonic; MFR Part No (none) -> P15.8KHCT-ND; Power W -> 1/10W; Tolerance % -> 1%
Connections:
- net +3.3V: no longer C29.1, L3.2, R14.2
- net +BATT: now also R1.1, R10.2, R11.2; no longer R10.1, R11.1
- net RADIO_EN: now also R1.2, U2.4 (~SHDN); no longer R1.1
- net at U4.4 (En): now also R11.1; no longer R11.2
- net at U3.4 (En): now also R10.1; no longer R10.2
- new net +1.8V: C29.1, L3.2, R14.2
Other:
- moved on the sheet: C17
