File: Electronics/RadioManager/Switch.sch (KiCad schematic (older format))
At the start: 28 parts, among them U1 KSZ8995FQI

Commit message: Load new 3d models
Parts:
- gave numbers to parts that had none: 11

Commit message: Add missing decoupling cap
Parts:
- added C30: C, ~, symbol C
- C22, C23: value C -> 33pF; Dielectric D -> NP0; Distributor Part No (none) -> 399-1055-6-ND; MFR Name (none) -> Kemet; MFR Part No (none) -> C0603C330J5GACTU; Voltage V -> 50V
- X1: Distributor Part No (none) -> 535-9847-1-ND; MFR Name (none) -> Abracon; MFR Part No (none) -> ABM7-25.000MHZ-D2Y-T
Connections:
- net +3.3V: now also C30.1
- net GND: now also C30.2

Commit message: Connect LEDs
Connections:
- net ACT1: now reaches U1.104 (LED1-2)
- net SPD1: now reaches U1.106 (LED1-0)
- net ACT2: now reaches U1.101 (LED2-2)
- net SPD2: now reaches U1.103 (LED2-0)
- net ACT3: now reaches U1.96 (LED3-2)
- net SPD3: now reaches U1.98 (LED3-0)
- net ACT4: now reaches U1.93 (LED4-2)
- net SPD4: now reaches U1.95 (LED4-0)
- net ACT5: now reaches U1.90 (LED5-2)
- net SPD5: now reaches U1.92 (LED5-0)
- no-connect marks 17 -> 22

Commit message: Swap tx/rx pairs for better routing
Connections:
- net RXM1: now also U1.8 (TXM1); no longer U1.5 (RXM1)
- net RXM2: now also U1.14 (TXM2); no longer U1.11 (RXM2)
- net RXM3: now also U1.23 (TXM3); no longer U1.20 (RXM3)
- net RXM4: now also U1.29 (TXM4); no longer U1.26 (RXM4)
- net RXM5: now also U1.36 (TXM5); no longer U1.33 (RXM5)
- net RXP1: now also U1.7 (TXP1); no longer U1.4 (RXP1)
- net RXP2: now also U1.13 (TXP2); no longer U1.10 (RXP2)
- net RXP3: now also U1.22 (TXP3); no longer U1.19 (RXP3)
- net RXP4: now also U1.28 (TXP4); no longer U1.25 (RXP4)
- net RXP5: now also U1.35 (TXP5); no longer U1.32 (RXP5)
- net TXM1: now also U1.5 (RXM1); no longer U1.8 (TXM1)
- net TXM2: now also U1.11 (RXM2); no longer U1.14 (TXM2)
- net TXM3: now also U1.20 (RXM3); no longer U1.23 (TXM3)
- net TXM4: now also U1.26 (RXM4); no longer U1.29 (TXM4)
- net TXM5: now also U1.33 (RXM5); no longer U1.36 (TXM5)
- net TXP1: now also U1.4 (RXP1); no longer U1.7 (TXP1)
- net TXP2: now also U1.10 (RXP2); no longer U1.13 (TXP2)
- net TXP3: now also U1.19 (RXP3); no longer U1.22 (TXP3)
- net TXP4: now also U1.25 (RXP4); no longer U1.28 (TXP4)
- net TXP5: now also U1.32 (RXP5); no longer U1.35 (TXP5)
Changed lines of the file:
@@
 Sheet 3 3
 Title ""
-Date "22 sep 2014"
+Date "3 oct 2014"
 Rev ""
 Comp ""
@@
 	1    0    0    -1
 $EndComp
-Text HLabel 10600 1200 2    60   Input ~ 0
+Text HLabel 10600 1400 2    60   Input ~ 0
 RXP1
-Text HLabel 10600 1300 2    60   Input ~ 0
+Text HLabel 10600 1500 2    60   Input ~ 0
 RXM1
-Text HLabel 10600 1400 2    60   Output ~ 0
+Text HLabel 10600 1200 2    60   Output ~ 0
 TXP1
-Text HLabel 10600 1500 2    60   Output ~ 0
+Text HLabel 10600 1300 2    60   Output ~ 0
 TXM1
-Text HLabel 10600 2300 2    60   Input ~ 0
+Text HLabel 10600 2500 2    60   Input ~ 0
 RXP2
-Text HLabel 10600 2400 2    60   Input ~ 0
+Text HLabel 10600 2600 2    60   Input ~ 0
 RXM2
-Text HLabel 10600 3500 2    60   Input ~ 0
+Text HLabel 10600 3700 2    60   Input ~ 0
 RXM3
-Text HLabel 10600 4600 2    60   Input ~ 0
+Text HLabel 10600 4800 2    60   Input ~ 0
 RXM4
-Text HLabel 10600 5800 2    60   Input ~ 0
+Text HLabel 10600 6000 2    60   Input ~ 0
 RXM5
-Text HLabel 10600 3400 2    60   Input ~ 0
+Text HLabel 10600 3600 2    60   Input ~ 0
 RXP3
-Text HLabel 10600 4500 2    60   Input ~ 0
+Text HLabel 10600 4700 2    60   Input ~ 0
 RXP4
-Text HLabel 10600 5700 2    60   Input ~ 0
+Text HLabel 10600 5900 2    60   Input ~ 0
 RXP5
-Text HLabel 10600 2500 2    60   Output ~ 0
+Text HLabel 10600 2300 2    60   Output ~ 0
 TXP2
-Text HLabel 10600 3600 2    60   Output ~ 0
+Text HLabel 10600 3400 2    60   Output ~ 0
 TXP3
-Text HLabel 10600 4700 2    60   Output ~ 0
+Text HLabel 10600 4500 2    60   Output ~ 0
 TXP4
-Text HLabel 10600 5900 2    60   Output ~ 0
+Text HLabel 10600 5700 2    60   Output ~ 0
 TXP5
-Text HLabel 10600 2600 2    60   Output ~ 0
+Text HLabel 10600 2400 2    60   Output ~ 0
 TXM2
-Text HLabel 10600 3700 2    60   Output ~ 0
+Text HLabel 10600 3500 2    60   Output ~ 0
 TXM3
-Text HLabel 10600 4800 2    60   Output ~ 0
+Text HLabel 10600 4600 2    60   Output ~ 0
 TXM4
-Text HLabel 10600 6000 2    60   Output ~ 0
+Text HLabel 10600 5800 2    60   Output ~ 0
 TXM5
 $Comp

Commit message: Resistor values
Parts:
- removed D2: DIODE, ~, symbol DIODE
- R4, R6, R7, R8, R9: Distributor Part No (none) -> RHM10KCGCT-ND; MFR Name (none) -> Rohm; MFR Part No (none) -> MCR03ERTJ103; Power W -> 1/10W; Tolerance % -> 5%
