File: Antennas/Crossed Dipole PCB/CrossedDipolePCB.kicad_pcb (KiCad board)
At the start: 2 copper layers, 25.8 x 25.8 mm, 1 part

Commit message: Update boards for fabrication
Other:
- rule pad_to_mask_clearance: 0 -> 0.0762
Changed lines of the file:
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@@
     (mod_text_size 1 1)
     (mod_text_width 0.15)
-    (pad_size 0.75 0.75)
-    (pad_drill 0)
-    (pad_to_mask_clearance 0)
-    (aux_axis_origin 0 0)
+    (pad_size 2.5 2.5)
+    (pad_drill 2.05)
+    (pad_to_mask_clearance 0.0762)
+    (aux_axis_origin 150 100)
     (visible_elements 7FFFFFFF)
     (pcbplotparams
-      (layerselection 3178497)
+      (layerselection 284196865)
       (usegerberextensions true)
       (excludeedgelayer true)
@@
       (viasonmask false)
       (mode 1)
-      (useauxorigin false)
+      (useauxorigin true)
       (hpglpennumber 1)
       (hpglpenspeed 20)
@@
       (plotinvisibletext false)
       (padsonsilk false)
-      (subtractmaskfromsilk false)
+      (subtractmaskfromsilk true)
       (outputformat 1)
       (mirror false)
-      (drillshape 1)
+      (drillshape 0)
       (scaleselection 1)
-      (outputdirectory ""))
+      (outputdirectory Gerber/))
   )
   (net 0 "")
@@
       (effects (font (size 1 1) (thickness 0.15)))
     )
+    (fp_arc (start 0 0) (end 1.438 2.49) (angle 150) (layer F.Mask) (width 0.91))
+    (fp_arc (start 0 0) (end -1.438 -2.49) (angle 150) (layer F.Mask) (width 0.91))
     (fp_arc (start 0 0) (end 1.438 2.49) (angle 150) (layer F.Cu) (width 0.75))
     (fp_arc (start 0 0) (end -1.438 -2.49) (angle 150) (layer F.Cu) (width 0.75))
@@
     (fp_circle (center 0 0) (end 2.75 0) (layer Dwgs.User) (width 0.5))
     (pad C thru_hole circle (at 0 0 315) (size 2.5 2.5) (drill 2.05)
-      (layers *.Mask F.Cu F.SilkS)
+      (layers *.Cu *.Mask F.SilkS)
       (net 3 N-000001)
     )
